File: Hardware/uSDX_V1_01-KICAD-files/SDR_SSB.kicad_pcb (KiCad board)
At the start: 2 copper layers, 97.8 x 97.8 mm, 87 parts, among them CON1 HEADPHONE, CON2 MIC/PTT, J1 CLK0, J2 CLK1, J3 CLK2, J4 Antenna, J5 DC 12V, Q1 BS170, Q2 BS170, Q3 BS170, Q4 BS170, SW1 L_Button, SW2 R_Button, SW3 Tune, U1 L7805CV, U2 ATMEGA328-PU, U3 RC1602A, U4 LM4562, U5 FST3253, U6 SI5351Module_2, U7 74ACT00, U8 LPF_M, Y1 20 Mhz

Commit message: updated HW design
Parts:
- removed C33, C34: 100nF, Capacitor_THT:C_Disc_D3.0mm_W2.0mm_P2.50mm
- removed J2: CLK1, Connector_PinHeader_2.54mm:PinHeader_1x02_P2.54mm_Vertical
- removed J3: CLK2, Connector_PinHeader_2.54mm:PinHeader_1x02_P2.54mm_Vertical
- removed J4: Antenna, SMA_EDGE:SMA_Samtec_SMA-J-P-X-ST-EM1_EdgeMount
- removed J5: DC 12V, digikey-footprints:PinHeader_1x2_P2.54mm_Drill1.02mm
- removed L2: 100uH, Inductor_THT:L_Axial_L5.3mm_D2.2mm_P2.54mm_Vertical_Vishay_IM-1
- removed REF** (x4): Pin_D1.0mm_L10.0mm, Connector_Pin:Pin_D1.0mm_L10.0mm
- removed SW3: Tune, USDX_V_1_01:RotaryEncoder_Alps_EC11E-Switch_Vertical_Modified_H20mm
- removed U2: ATMEGA328-PU, Package_DIP:DIP-28_W7.62mm_Socket_LongPads
- removed Y1: 20 Mhz, Crystal:Crystal_HC49-U_Vertical
- added C29: 100nF, Capacitor_SMD:C_0805_2012Metric_Pad1.18x1.45mm_HandSolder, F.Cu at (121.9, -350.5)
- added C30: 10nF, Capacitor_SMD:C_0805_2012Metric_Pad1.18x1.45mm_HandSolder, F.Cu at (192.8, -245.5)
- added C31: 100nF, Capacitor_SMD:C_0805_2012Metric_Pad1.18x1.45mm_HandSolder, F.Cu at (167.6, -238.8)
- added D2: 1N4148W, Diode_SMD:D_SOD-123, F.Cu at (19.1, -214.6)
- added D3: 1N4148W, Diode_SMD:D_SOD-123, F.Cu at (27.9, -208.3)
- added Y2: 20 Mhz, Crystal:Crystal_HC49-U_Vertical, F.Cu at (149.9, -223.5)
- C1: footprint Capacitor_THT:CP_Radial_D5.0mm_P2.50mm -> Capacitor_SMD:CP_Elec_5x5.8
- C10, C19: value 100nF -> 10nF; footprint Capacitor_THT:C_Disc_D3.0mm_W2.0mm_P2.50mm -> Capacitor_SMD:C_0805_2012Metric_Pad1.18x1.45mm_HandSolder
- C11: value 10nF -> 10uF/16V; footprint Capacitor_THT:C_Disc_D3.0mm_W2.0mm_P2.50mm -> Capacitor_SMD:CP_Elec_4x4.5
- C12, C14, C17, C18, C2, C27, C3, C6, C8: footprint Capacitor_THT:C_Disc_D3.0mm_W2.0mm_P2.50mm -> Capacitor_SMD:C_0805_2012Metric_Pad1.18x1.45mm_HandSolder
- C13: value 100nF -> 33pF; footprint Capacitor_THT:C_Disc_D3.0mm_W2.0mm_P2.50mm -> Capacitor_SMD:C_0805_2012Metric_Pad1.18x1.45mm_HandSolder
- C15: value 1nF -> 10nF; footprint Capacitor_THT:C_Disc_D3.0mm_W2.0mm_P2.50mm -> Capacitor_SMD:C_0805_2012Metric_Pad1.18x1.45mm_HandSolder
- C16: value 1nF -> 100nF; footprint Capacitor_THT:C_Disc_D3.0mm_W2.0mm_P2.50mm -> Capacitor_SMD:C_0805_2012Metric_Pad1.18x1.45mm_HandSolder
- C20: value 100nF -> 470nF; footprint Capacitor_THT:C_Disc_D3.0mm_W2.0mm_P2.50mm -> Capacitor_SMD:C_0805_2012Metric_Pad1.18x1.45mm_HandSolder
- C21: value 10nF -> 470nF; footprint Capacitor_THT:C_Disc_D3.0mm_W2.0mm_P2.50mm -> Capacitor_SMD:C_0805_2012Metric_Pad1.18x1.45mm_HandSolder
- C22: value 470nF -> 100nF; footprint Capacitor_THT:C_Disc_D3.0mm_W2.0mm_P2.50mm -> Capacitor_SMD:C_0805_2012Metric_Pad1.18x1.45mm_HandSolder
- C23: value 470nF -> 1nF; footprint Capacitor_THT:C_Disc_D3.0mm_W2.0mm_P2.50mm -> Capacitor_SMD:C_0805_2012Metric_Pad1.18x1.45mm_HandSolder
- C24: value 10nF -> 1nF; footprint Capacitor_THT:C_Disc_D3.0mm_W2.0mm_P2.50mm -> Capacitor_SMD:C_0805_2012Metric_Pad1.18x1.45mm_HandSolder
- C25, C26: value 10nF -> 100nF; footprint Capacitor_THT:C_Disc_D3.0mm_W2.0mm_P2.50mm -> Capacitor_SMD:C_0805_2012Metric_Pad1.18x1.45mm_HandSolder
- C28: value 33pF -> 100nF; footprint Capacitor_THT:C_Disc_D3.0mm_W2.0mm_P2.50mm -> Capacitor_SMD:C_0805_2012Metric_Pad1.18x1.45mm_HandSolder
- C4: value 10uF -> 100nF; footprint Capacitor_THT:CP_Radial_D4.0mm_P2.00mm -> Capacitor_SMD:C_0805_2012Metric_Pad1.18x1.45mm_HandSolder
- C5: footprint Capacitor_THT:CP_Radial_D4.0mm_P2.00mm -> Capacitor_SMD:C_0805_2012Metric_Pad1.18x1.45mm_HandSolder
- C7: value 100nF -> 10uF; footprint Capacitor_THT:C_Disc_D3.0mm_W2.0mm_P2.50mm -> Capacitor_SMD:C_0805_2012Metric_Pad1.18x1.45mm_HandSolder
- C9: value 10uF/16V -> 10nF; footprint Capacitor_THT:CP_Radial_D4.0mm_P2.00mm -> Capacitor_SMD:C_0805_2012Metric_Pad1.18x1.45mm_HandSolder
- CON1, CON2: footprint digikey-footprints:Headphone_Jack_3.5mm_SJ1-3523N -> Connector_Audio:Jack_3.5mm_CUI_SJ1-3533NG_Horizontal
- D1: footprint Diode_THT:D_A-405_P2.54mm_Vertical_AnodeUp -> Diode_THT:D_DO-41_SOD81_P10.16mm_Horizontal
- J1: value CLK0 -> DC 12V; footprint Connector_PinHeader_2.54mm:PinHeader_1x02_P2.54mm_Vertical -> Connector_BarrelJack:BarrelJack_CUI_PJ-036AH-SMT_Horizontal
- L3: value T37_2(10T) -> 100uH; footprint Inductor_THT:L_Toroid_Vertical_L10.0mm_W5.0mm_P5.08mm -> Inductor_THT:L_Axial_L5.3mm_D2.2mm_P2.54mm_Vertical_Vishay_IM-1
- Q1, Q2, Q3, Q4: footprint Package_TO_SOT_THT:TO-92L_HandSolder -> Package_TO_SOT_THT:TO-92_Inline
- R1, R24, R3: value 10k -> 1k; footprint Resistor_THT:R_Axial_DIN0204_L3.6mm_D1.6mm_P1.90mm_Vertical -> Resistor_SMD:R_0805_2012Metric_Pad1.20x1.40mm_HandSolder
- R10, R11, R12, R19, R2, R20: footprint Resistor_THT:R_Axial_DIN0204_L3.6mm_D1.6mm_P1.90mm_Vertical -> Resistor_SMD:R_0805_2012Metric_Pad1.20x1.40mm_HandSolder
- R13, R14, R15: value 10k -> 100; footprint Resistor_THT:R_Axial_DIN0204_L3.6mm_D1.6mm_P1.90mm_Vertical -> Resistor_SMD:R_0805_2012Metric_Pad1.20x1.40mm_HandSolder
- R16: value 3.3k -> 100; footprint Resistor_THT:R_Axial_DIN0204_L3.6mm_D1.6mm_P1.90mm_Vertical -> Resistor_SMD:R_0805_2012Metric_Pad1.20x1.40mm_HandSolder
- R17: value 1k -> 82k; footprint Resistor_THT:R_Axial_DIN0204_L3.6mm_D1.6mm_P1.90mm_Vertical -> Resistor_SMD:R_0805_2012Metric_Pad1.20x1.40mm_HandSolder
- R18: value 10k -> 82k; footprint Resistor_THT:R_Axial_DIN0204_L3.6mm_D1.6mm_P1.90mm_Vertical -> Resistor_SMD:R_0805_2012Metric_Pad1.20x1.40mm_HandSolder
- R21, R25: value 1k -> 10k; footprint Resistor_THT:R_Axial_DIN0204_L3.6mm_D1.6mm_P1.90mm_Vertical -> Resistor_SMD:R_0805_2012Metric_Pad1.20x1.40mm_HandSolder
- R22: value 1k-1/2W -> 10k; footprint Resistor_THT:R_Axial_DIN0204_L3.6mm_D1.6mm_P2.54mm_Vertical -> Resistor_SMD:R_0805_2012Metric_Pad1.20x1.40mm_HandSolder
- R23: value 470 -> 3.3k; footprint Resistor_THT:R_Axial_DIN0204_L3.6mm_D1.6mm_P1.90mm_Vertical -> Resistor_SMD:R_0805_2012Metric_Pad1.20x1.40mm_HandSolder
- R4, R5, R8, R9: value 100 -> 10k; footprint Resistor_THT:R_Axial_DIN0204_L3.6mm_D1.6mm_P1.90mm_Vertical -> Resistor_SMD:R_0805_2012Metric_Pad1.20x1.40mm_HandSolder
- R6: value 82k -> 1k; footprint Resistor_THT:R_Axial_DIN0204_L3.6mm_D1.6mm_P1.90mm_Vertical -> Resistor_SMD:R_0805_2012Metric_Pad1.20x1.40mm_HandSolder
- R7: value 82k -> 470; footprint Resistor_THT:R_Axial_DIN0204_L3.6mm_D1.6mm_P1.90mm_Vertical -> Resistor_SMD:R_0805_2012Metric_Pad1.20x1.40mm_HandSolder; moved to B.Cu
- RV1: footprint Potentiometer_THT:Potentiometer_Piher_PT-10-V10_Vertical -> Potentiometer_THT:Potentiometer_Piher_PT-6-V_Vertical
- SW1, SW2: footprint Button_Switch_THT:SW_PUSH_6mm -> Button_Switch_THT:SW_PUSH-12mm
- U1: value L7805CV -> Si5351A-B-GT; footprint digikey-footprints:TO-220-3 -> Package_SO:MSOP-10_3x3mm_P0.5mm
- U3: value RC1602A -> L7805CV; footprint Display:WC1602A -> Package_TO_SOT_SMD:TO-252-3_TabPin4
- U4: value LM4562 -> FST3253; footprint Package_DIP:DIP-8_W7.62mm_LongPads -> Package_SO:SOIC-16_4.55x10.3mm_P1.27mm
- U5: value FST3253 -> LM4562; footprint Package_SO:SOIC-16_4.55x10.3mm_P1.27mm -> Package_SO:SOIC-8_3.9x4.9mm_P1.27mm
- U6: value SI5351Module_2 -> 74ACT00; footprint VFO_footprint:SI5351 Module -> Package_SO:SOIC-14_3.9x8.7mm_P1.27mm
- U7: value 74ACT00 -> RC1602A; footprint Package_DIP:DIP-14_W7.62mm_LongPads -> Display:WC1602A
- U8: value LPF_M -> ATMEGA328-PU; footprint QRP_LPF:LPF_M -> Package_QFP:TQFP-32_7x7mm_P0.8mm
- moved Q4 246.0 mm to (341.6, -177.8), turned to 0 degrees
- moved C26 240.1 mm to (326.4, -293.4)
- moved R12 234.7 mm to (336.6, -165.1), turned to 0 degrees
- moved C24 231.2 mm to (313.7, -301.0), turned to 0 degrees
- moved Q2 229.9 mm to (323.9, -179.1), turned to 0 degrees
- moved R14 224.5 mm to (317.5, -278.1)
- moved R21 221.3 mm to (316.2, -269.3)
- moved R20 221.1 mm to (337.8, -289.6)
- moved C17 219.9 mm to (328.9, -281.9), turned to 0 degrees
- moved R19 218.5 mm to (336.6, -299.7), turned to 0 degrees
- moved R13 217.1 mm to (317.5, -283.2), turned to 0 degrees
- moved R8 214.9 mm to (-2.54, -377.2), turned to 0 degrees
- moved C10 214.8 mm to (294.6, -147.3)
- moved Q3 214.0 mm to (308.6, -177.8), turned to 0 degrees
- moved C16 203.5 mm to (1.27, -364.5)
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Connections:
- C10 pad 1: Net-(C10-Pad1) -> GNDPWR
- C10 pad 2: Net-(C10-Pad2) -> PB0
- C11 pad 1: Net-(C10-Pad1) -> Net-(C11-Pad1)
- C11 pad 2: GNDPWR -> Net-(C11-Pad2)
- C12 pad 2: Net-(C12-Pad2) -> RF_SIGNAL
- C13 pad 1: Net-(C13-Pad1) -> Net-(C12-Pad1)
- C13 pad 2: Net-(C13-Pad2) -> GNDPWR
- C14 pad 1: GNDPWR -> +5V
- C14 pad 2: Net-(C14-Pad2) -> GNDPWR
- C15 pad 1: Net-(C15-Pad1) -> PB4
- C15 pad 2: Net-(C12-Pad1) -> GNDPWR
- C16 pad 1: Net-(C16-Pad1) -> PB4
- C16 pad 2: Net-(C13-Pad1) -> PC2
- C17 pad 2: Net-(C17-Pad2) -> 90_deg
- C18 pad 1: GNDPWR -> 0_deg
- C18 pad 2: Net-(C18-Pad2) -> GNDPWR
- C19 pad 1: +5V -> Net-(C19-Pad1)
- C20 pad 1: Net-(C20-Pad1) -> GNDPWR
- C20 pad 2: GNDPWR -> 180_deg
- C21 pad 1: Net-(C21-Pad1) -> 270_deg
- C21 pad 2: Net-(C21-Pad2) -> GNDPWR
- C22 pad 1: Net-(C22-Pad1) -> +5V
- C23 pad 2: GNDPWR -> Net-(C23-Pad2)
- C25 pad 1: Net-(C25-Pad1) -> +12V
- C26 pad 1: Net-(C26-Pad1) -> Net-(C24-Pad2)
- C26 pad 2: GNDPWR -> I
- C27 pad 1: Net-(C27-Pad1) -> Net-(C23-Pad2)
- C27 pad 2: Net-(C27-Pad2) -> Q
- C28 pad 2: Net-(C27-Pad1) -> AREF
- C3 pad 1: +5V -> GNDPWR
- C3 pad 2: GNDPWR -> Net-(C3-Pad2)
- C4 pad 1: +5V -> Net-(C4-Pad1)
- C5 pad 1: Net-(C5-Pad1) -> Net-(C4-Pad1)
- C6 pad 1: Net-(C5-Pad1) -> +5V
- C7 pad 1: Net-(C7-Pad1) -> +5V
- C8 pad 1: Net-(C5-Pad1) -> Net-(C8-Pad1)
- C9 pad 2: Net-(C9-Pad2) -> F_IN
- J1 pad 1: Net-(J1-Pad1) -> Net-(D1-Pad1)
- L1 pad 1: +5V -> Net-(C4-Pad1)
- L1 pad 2: Net-(C5-Pad1) -> +5V
- L3 pad 1: +12V -> +5V
- L3 pad 2: Net-(C27-Pad1) -> AVCC
- Q1 pad 1: Net-(C27-Pad2) -> RF_SIGNAL
- Q1 pad 2: Net-(C25-Pad1) -> PB0
- Q1 pad 3: Net-(C21-Pad2) -> F_IN
- Q2 pad 1: Net-(C27-Pad1) -> Net-(C12-Pad1)
- Q2 pad 2: Net-(C24-Pad1) -> CTRL_OUT
- Q3 pad 1: Net-(C27-Pad1) -> Net-(C12-Pad1)
- Q3 pad 2: Net-(C24-Pad1) -> CTRL_OUT
- Q4 pad 1: Net-(C27-Pad1) -> Net-(C12-Pad1)
- Q4 pad 2: Net-(C24-Pad1) -> CTRL_OUT
- R1 pad 1: +5V -> Net-(C3-Pad2)
- R1 pad 2: Net-(C20-Pad1) -> RS
- R10 pad 1: Net-(C12-Pad2) -> AREF
- R10 pad 2: Net-(C14-Pad2) -> PC2
- R11 pad 1: GNDPWR -> PC2
- R11 pad 2: Net-(C12-Pad2) -> GNDPWR
- R12 pad 1: Net-(C13-Pad2) -> TX_CTRL_1
- R12 pad 2: Net-(C14-Pad2) -> Net-(C19-Pad1)
- R13 pad 1: GNDPWR -> 180_deg
- R13 pad 2: Net-(C13-Pad2) -> Net-(C24-Pad1)
- R14 pad 1: Net-(C24-Pad1) -> 90_deg
- R14 pad 2: Net-(C26-Pad1) -> Net-(R14-Pad2)
- R15 pad 1: Net-(C26-Pad1) -> 0_deg
- R15 pad 2: Net-(R15-Pad2) -> Net-(C23-Pad1)
- R16 pad 1: Net-(R16-Pad1) -> 270_deg
- R16 pad 2: +5V -> Net-(R16-Pad2)
- R17 pad 1: Net-(R17-Pad1) -> Net-(C23-Pad1)
- R17 pad 2: +5V -> Net-(C23-Pad2)
- R18 pad 1: Net-(R18-Pad1) -> Net-(C24-Pad1)
- R18 pad 2: GNDPWR -> Net-(C24-Pad2)
- R19 pad 1: Net-(C10-Pad2) -> I
- R19 pad 2: GNDPWR -> AREF
- R2 pad 1: Net-(C20-Pad1) -> Net-(C3-Pad2)
- R2 pad 2: Net-(C21-Pad1) -> SCL
- R20 pad 1: Net-(C14-Pad2) -> GNDPWR
- R20 pad 2: Net-(C10-Pad2) -> I
- R21 pad 1: Net-(R21-Pad1) -> Q
- R21 pad 2: GNDPWR -> AREF
- R22 pad 1: +12V -> GNDPWR
- R22 pad 2: Net-(R22-Pad2) -> Q
- R23 pad 2: Net-(C9-Pad1) -> +5V
- R24 pad 1: Net-(C7-Pad1) -> Net-(R24-Pad1)
- R24 pad 2: Net-(C10-Pad1) -> +5V
- R25 pad 1: Net-(C21-Pad2) -> BUT_STATE
- R3 pad 1: Net-(C20-Pad1) -> F_IN
- R4 pad 1: Net-(C17-Pad2) -> +5V
- R4 pad 2: Net-(C15-Pad1) -> Net-(C8-Pad1)
- R5 pad 1: Net-(C18-Pad2) -> Net-(C8-Pad1)
- R5 pad 2: Net-(R5-Pad2) -> GNDPWR
- R6 pad 1: Net-(C15-Pad1) -> Net-(C8-Pad1)
- R6 pad 2: Net-(C12-Pad1) -> Net-(C9-Pad1)
- R7 pad 1: Net-(C16-Pad1) -> HP_OUT
- R7 pad 2: Net-(C13-Pad1) -> Net-(C11-Pad1)
- R8 pad 1: Net-(C22-Pad1) -> AVCC
- R8 pad 2: Net-(C16-Pad1) -> PB4
- R9 pad 1: Net-(C23-Pad1) -> Net-(C19-Pad1)
- R9 pad 2: Net-(R9-Pad2) -> CTRL_OUT
- RV1 pad 1: Net-(C5-Pad1) -> +5V
- RV1 pad 3: Net-(R21-Pad1) -> GNDPWR
- SW1 pad 1: Net-(R18-Pad1) -> BUT_STATE
- SW1 pad 2: Net-(R16-Pad1) -> Net-(R23-Pad1)
- SW2 pad 1: Net-(R18-Pad1) -> BUT_STATE
- SW2 pad 2: Net-(R17-Pad1) -> Net-(R24-Pad1)
- U1 pad 1: +12V -> Net-(C3-Pad2)
- U1 pad 2: GNDPWR -> Net-(U1-Pad2)
- U1 pad 3: +5V -> Net-(U1-Pad3)
- U3 pad 1: GNDPWR -> +12V
- U3 pad 2: Net-(C5-Pad1) -> GNDPWR
- U3 pad 3: Net-(RV1-Pad2) -> Net-(C4-Pad1)
- U3 pad 4: Net-(U2-Pad27) -> (no net)
- U4 pad 1: Net-(C13-Pad1) -> +5V
- U4 pad 2: Net-(C16-Pad1) -> CLK_1
- U4 pad 3: Net-(R9-Pad2) -> Net-(U4-Pad3)
- U4 pad 4: GNDPWR -> Net-(U4-Pad4)
- U4 pad 5: Net-(R5-Pad2) -> Net-(U4-Pad5)
- U4 pad 6: Net-(C15-Pad1) -> Net-(U4-Pad6)
- U4 pad 7: Net-(C12-Pad1) -> GNDPWR
- U4 pad 8: +12V -> GNDPWR
- U5 pad 1: Net-(U5-Pad1) -> Net-(C23-Pad2)
- U5 pad 2: Net-(J2-Pad1) -> Net-(C23-Pad1)
- U5 pad 3: Net-(U5-Pad3) -> Net-(R16-Pad2)
- U5 pad 4: Net-(U5-Pad4) -> GNDPWR
- U5 pad 5: Net-(U5-Pad5) -> Net-(R14-Pad2)
- U5 pad 6: Net-(U5-Pad6) -> Net-(C24-Pad1)
- U5 pad 7: Net-(U5-Pad7) -> Net-(C24-Pad2)
- U5 pad 8: GNDPWR -> +12V
- U6 pad 1: +5V -> CLK_2
- U6 pad 2: GNDPWR -> Net-(U6-Pad2)
- U6 pad 3: Net-(U2-Pad27) -> Net-(U6-Pad3)
- U6 pad 4: Net-(U2-Pad28) -> Net-(U6-Pad3)
- U6 pad 5: Net-(U6-Pad5) -> Net-(U6-Pad3)
- U6 pad 7: Net-(U6-Pad7) -> GNDPWR
- U7 pad 1: Net-(U7-Pad1) -> GNDPWR
- U7 pad 10: Net-(C25-Pad1) -> Net-(U7-Pad10)
- U7 pad 11: Net-(U7-Pad11) -> DB4
- U7 pad 12: +5V -> DB5
- U7 pad 13: +5V -> DB6
- U7 pad 14: +5V -> DB7
- U7 pad 2: Net-(J3-Pad1) -> +5V
- U7 pad 3: Net-(U7-Pad3) -> Net-(RV1-Pad2)
- U7 pad 4: Net-(U7-Pad3) -> RS
- U7 pad 5: Net-(U7-Pad3) -> GNDPWR
- U7 pad 6: Net-(C24-Pad2) -> E
- U7 pad 7: GNDPWR -> Net-(U7-Pad7)
- U7 pad 8: Net-(U7-Pad1) -> Net-(U7-Pad8)
- U7 pad 9: Net-(C25-Pad1) -> Net-(U7-Pad9)
- U8 pad 1: Net-(C27-Pad2) -> Net-(U8-Pad1)
- U8 pad 2: Net-(C27-Pad2) -> DB4
- U8 pad 3: GNDPWR -> DB5
- U8 pad 4: GNDPWR -> DB6
- U8 pad 5: Net-(J4-Pad1) -> DB7
- U8 pad 6: Net-(J4-Pad1) -> E
- U8 pad 7: GNDPWR -> +5V
Routing:
- net +5V: track 235.1 -> 0.00 mm, vias 4 -> 0
- net +12V: track 177.0 -> 0.00 mm, vias 1 -> 0
- net Net-(C25-Pad1): track 150.3 -> 0.00 mm, vias 3 -> 0
- net Net-(C5-Pad1): track 144.3 -> 0.00 mm
- net Net-(U2-Pad27): track 132.0 -> 0.00 mm, vias 2 -> 0
- net Net-(C14-Pad2): track 107.2 -> 0.00 mm, vias 2 -> 0
- net Net-(R18-Pad1): track 99.7 -> 0.00 mm, vias 2 -> 0
- net Net-(C18-Pad2): track 97.4 -> 0.00 mm, vias 2 -> 0
- net Net-(J3-Pad1): track 92.4 -> 0.00 mm, vias 1 -> 0
- net Net-(C13-Pad2): track 89.0 -> 0.00 mm, vias 1 -> 0
- net Net-(C12-Pad2): track 87.5 -> 0.00 mm
- net Net-(C21-Pad2): track 87.2 -> 0.00 mm
- net Net-(U2-Pad28): track 84.8 -> 0.00 mm
- net Net-(R15-Pad2): track 82.1 -> 0.00 mm
- net Net-(R23-Pad1): track 79.7 -> 0.00 mm
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- removed copper zone on B.Cu, net GNDPWR
- removed copper zone on F.Cu, net GNDPWR
Other:
- board outline removed
- board text removed: "+12V"
- board text removed: "1"
- board text removed: "16"
- board text removed: "All Mode SDR HF Transceiver"
- board text removed: "Design&Firmware: PE1NNZ"
- board text removed: "GND"
- board text removed: "Max"
- board text removed: "Min"
- board text removed: "PCB Ver 1.01 : WB2CBA"
- board text removed: "SMA"
- board text removed: "uSDX"
- board text removed: "uSDX - SDR HF TRX"
