File: Hardware/uSDX_V1_01-KICAD-files/SDR_SSB.sch (KiCad schematic (older format))
At the start: 90 parts, among them CON1 HEADPHONE, CON2 MIC/PTT, J4 Antenna, U2 ATMEGA328-PU, U3 RC1602A, U8 LPF_M, Y1 20 Mhz

Commit message: updated component footprints
Parts:
- C1: renamed from C?; footprint Capacitor_THT:CP_Radial_D5.0mm_P2.50mm -> Capacitor_SMD:CP_Elec_5x5.8; Link (none) -> https://ro.mouser.com/ProductDetail/Panasonic/EEE-FK1C101SR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; Mfr. No. (none) -> EEE-FK1C101SR
- C10, C19: renamed from C?; footprint (none) -> Capacitor_SMD:C_0805_2012Metric_Pad1.18x1.45mm_HandSolder; Link (none) -> https://ro.mouser.com/ProductDetail/Wurth-Elektronik/885382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; Mfr. No. (none) -> 885382207009
- C11: renamed from C9; footprint Capacitor_THT:CP_Radial_D4.0mm_P2.00mm -> Capacitor_SMD:CP_Elec_4x4.5; Link (none) -> https://ro.mouser.com/ProductDetail/Nichicon/UCQ1C100MCL1GB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; Mfr. No. (none) -> UCQ1C100MCL1GB
- C12, C3: renamed from C?; footprint (none) -> Capacitor_SMD:C_0805_2012Metric_Pad1.18x1.45mm_HandSolder; Link (none) -> https://ro.mouser.com/ProductDetail/Wurth-Elektronik/885012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; Mfr. No. (none) -> 885012207072
- C13: renamed from C?; footprint (none) -> Capacitor_SMD:C_0805_2012Metric_Pad1.18x1.45mm_HandSolder; Link (none) -> https://ro.mouser.com/ProductDetail/KEMET/C0805C330J5GACTU?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; Mfr. No. (none) -> C0805C330J5GACTU
- C14, C2, C22, C25, C26, C27, C28, C4, C8: renamed from C?; footprint Capacitor_THT:C_Disc_D3.0mm_W2.0mm_P2.50mm -> Capacitor_SMD:C_0805_2012Metric_Pad1.18x1.45mm_HandSolder; Link (none) -> https://ro.mouser.com/ProductDetail/Wurth-Elektronik/885012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; Mfr. No. (none) -> 885012207072
- C15: renamed from C11; footprint Capacitor_THT:C_Disc_D3.0mm_W2.0mm_P2.50mm -> Capacitor_SMD:C_0805_2012Metric_Pad1.18x1.45mm_HandSolder; Link (none) -> https://ro.mouser.com/ProductDetail/Wurth-Elektronik/885382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; Mfr. No. (none) -> 885382207009
- C16: renamed from C10; footprint Capacitor_THT:C_Disc_D3.0mm_W2.0mm_P2.50mm -> Capacitor_SMD:C_0805_2012Metric_Pad1.18x1.45mm_HandSolder; Link (none) -> https://ro.mouser.com/ProductDetail/Wurth-Elektronik/885012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; Mfr. No. (none) -> 885012207072
- C17, C18: renamed from C?; footprint Capacitor_THT:C_Disc_D3.0mm_W2.0mm_P2.50mm -> Capacitor_SMD:C_0805_2012Metric_Pad1.18x1.45mm_HandSolder; Link (none) -> https://ro.mouser.com/ProductDetail/Samsung-Electro-Mechani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; Mfr. No. (none) -> CL21B474KAFNNNG
- C20, C21: renamed from C?; footprint Capacitor_THT:C_Disc_D3.0mm_W2.0mm_P2.50mm -> Capacitor_SMD:C_0805_2012Metric_Pad1.18x1.45mm_HandSolder; Link (none) -> https://ro.mouser.com/ProductDetail/Samsung-Electro-Mechani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; Mfr. No (none) -> 885012207070; Mfr. No. (none) -> CL21B474KAFNNNG
- C23, C24: renamed from C?; footprint Capacitor_THT:C_Disc_D3.0mm_W2.0mm_P2.50mm -> Capacitor_SMD:C_0805_2012Metric_Pad1.18x1.45mm_HandSolder; Link (none) -> https://ro.mouser.com/ProductDetail/710-885012007040; Mfr. No. (none) -> 885012007040
- C29: renamed from C8; footprint Capacitor_THT:C_Disc_D3.0mm_W2.0mm_P2.50mm -> Capacitor_SMD:C_0805_2012Metric_Pad1.18x1.45mm_HandSolder; Link (none) -> https://ro.mouser.com/ProductDetail/Wurth-Elektronik/885012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; Mfr. No. (none) -> 885012207072
- C30: renamed from C?; footprint Capacitor_THT:C_Disc_D3.0mm_W2.0mm_P2.50mm -> Capacitor_SMD:C_0805_2012Metric_Pad1.18x1.45mm_HandSolder; Link (none) -> https://ro.mouser.com/ProductDetail/Wurth-Elektronik/885382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; Mfr. No. (none) -> 885382207009
- C31: renamed from C?; value C -> 100nF; footprint (none) -> Capacitor_SMD:C_0805_2012Metric_Pad1.18x1.45mm_HandSolder; Link (none) -> https://ro.mouser.com/ProductDetail/Wurth-Elektronik/885012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; Mfr. No. (none) -> 885012207072
- C5: renamed from C?; footprint Capacitor_THT:CP_Radial_D4.0mm_P2.00mm -> Capacitor_SMD:C_0805_2012Metric_Pad1.18x1.45mm_HandSolder; Link (none) -> https://ro.mouser.com/ProductDetail/Nichicon/UCQ1C100MCL1GB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; Mfr. No. (none) -> UCQ1C100MCL1GB
- C6: footprint Capacitor_THT:C_Disc_D3.0mm_W2.0mm_P2.50mm -> Capacitor_SMD:C_0805_2012Metric_Pad1.18x1.45mm_HandSolder; Link (none) -> https://ro.mouser.com/ProductDetail/Wurth-Elektronik/885012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; Mfr. No. (none) -> 885012207072
- C7: renamed from C5; footprint Capacitor_THT:CP_Radial_D4.0mm_P2.00mm -> Capacitor_SMD:C_0805_2012Metric_Pad1.18x1.45mm_HandSolder; Link (none) -> https://ro.mouser.com/ProductDetail/Nichicon/UCQ1C100MCL1GB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; Mfr. No. (none) -> UCQ1C100MCL1GB
- C9: renamed from C?; footprint Capacitor_THT:C_Disc_D3.0mm_W2.0mm_P2.50mm -> Capacitor_SMD:C_0805_2012Metric_Pad1.18x1.45mm_HandSolder; Link (none) -> https://ro.mouser.com/ProductDetail/Wurth-Elektronik/885382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; Mfr. No. (none) -> 885382207009; Mfr.No. (none) -> C0603C103K3TACAUTO
- CON1, CON2: footprint digikey-footprints:Headphone_Jack_3.5mm_SJ1-3523N -> Connector_Audio:Jack_3.5mm_CUI_SJ1-3533NG_Horizontal; Link (none) -> https://ro.mouser.com/ProductDetail/Kycon/STX-3150-3C-1?qs=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; Mfr. No. (none) -> STX-3150-3C-1
- D1: renamed from D?; footprint Diode_THT:D_A-405_P2.54mm_Vertical_AnodeUp -> Diode_THT:D_DO-41_SOD81_P10.16mm_Horizontal; Link (none) -> https://ro.mouser.com/ProductDetail/Taiwan-Semiconductor/1N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; Mfr. No. (none) -> 1N4007G A0G
- D2, D3: renamed from D?; Link (none) -> https://ro.mouser.com/ProductDetail/Panjit/1N4148W_R2_00001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; Mfr. No. (none) -> 1N4148W_R2_00001
- J1: renamed from J?; footprint digikey-footprints:PinHeader_1x2_P2.54mm_Drill1.02mm -> Connector_BarrelJack:BarrelJack_CUI_PJ-036AH-SMT_Horizontal; Link (none) -> https://ro.mouser.com/ProductDetail/Switchcraft/RASM722BKZ?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; Mfr. No. (none) -> RASM722BKZ
- J2: renamed from J4; Link (none) -> https://ro.mouser.com/ProductDetail/Linx-Technologies/CONSM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; Mfr. No. (none) -> CONSMA002-SMD-G-T
- L1: Link (none) -> https://ro.mouser.com/ProductDetail/Coilcraft/MSS6122-104ML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; Mfr. No. (none) -> MSS6122-104MLC
- L2: renamed from L?; value T37_2(10T) -> T50_2(9T)
- L3: renamed from L2; Link (none) -> https://ro.mouser.com/ProductDetail/TDK/VLS3010CX-101M-1?qs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; Mfr. No. (none) -> VLS3010CX-101M-1
- Q1, Q2, Q3, Q4: renamed from Q?; Link (none) -> https://ro.mouser.com/ProductDetail/onsemi-Fairchild/BS170-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; Mfr. No. (none) -> BS170-D75Z
- R1, R2, R3: renamed from R?; footprint (none) -> Resistor_SMD:R_0805_2012Metric_Pad1.20x1.40mm_HandSolder; Link (none) -> https://ro.mouser.com/ProductDetail/YAGEO/RC0805FR-071KL?qs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; Mfr. No. (none) -> RC0805FR-071KL
- R10: renamed from R20; footprint Resistor_THT:R_Axial_DIN0204_L3.6mm_D1.6mm_P1.90mm_Vertical -> Resistor_SMD:R_0805_2012Metric_Pad1.20x1.40mm_HandSolder; Link (none) -> https://ro.mouser.com/ProductDetail/Vishay-Dale/CRCW080510K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; Mfr. No. (none) -> CRCW080510K0FKEAC
- R11: renamed from R19; footprint Resistor_THT:R_Axial_DIN0204_L3.6mm_D1.6mm_P1.90mm_Vertical -> Resistor_SMD:R_0805_2012Metric_Pad1.20x1.40mm_HandSolder; Link (none) -> https://ro.mouser.com/ProductDetail/Vishay-Dale/CRCW080510K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; Mfr. No. (none) -> CRCW080510K0FKEAC
- R12, R9: renamed from R?; footprint (none) -> Resistor_SMD:R_0805_2012Metric_Pad1.20x1.40mm_HandSolder; Link (none) -> https://ro.mouser.com/ProductDetail/Vishay-Dale/CRCW080510K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; Mfr. No. (none) -> CRCW080510K0FKEAC
- R13, R14, R15, R16: renamed from R?; footprint Resistor_THT:R_Axial_DIN0204_L3.6mm_D1.6mm_P1.90mm_Vertical -> Resistor_SMD:R_0805_2012Metric_Pad1.20x1.40mm_HandSolder; Link (none) -> https://ro.mouser.com/ProductDetail/Bourns/CRM0805-FX-1000E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; Mfr. No. (none) -> CRM0805-FX-1000ELF
- R17, R18: renamed from R?; footprint Resistor_THT:R_Axial_DIN0204_L3.6mm_D1.6mm_P1.90mm_Vertical -> Resistor_SMD:R_0805_2012Metric_Pad1.20x1.40mm_HandSolder; Link (none) -> https://ro.mouser.com/ProductDetail/YAGEO/RC0805FR-0782KL?q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; Mfr. No. (none) -> RC0805FR-0782KL
- R19, R20, R21, R22, R25, R4, R5: renamed from R?; footprint Resistor_THT:R_Axial_DIN0204_L3.6mm_D1.6mm_P1.90mm_Vertical -> Resistor_SMD:R_0805_2012Metric_Pad1.20x1.40mm_HandSolder; Link (none) -> https://ro.mouser.com/ProductDetail/Vishay-Dale/CRCW080510K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; Mfr. No. (none) -> CRCW080510K0FKEAC
- R23: renamed from R?; footprint Resistor_THT:R_Axial_DIN0204_L3.6mm_D1.6mm_P1.90mm_Vertical -> Resistor_SMD:R_0805_2012Metric_Pad1.20x1.40mm_HandSolder; Link (none) -> https://ro.mouser.com/ProductDetail/YAGEO/AC0805FR-7W3K3L?q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; Mfr. No. (none) -> AC0805FR-7W3K3L
- R24, R6: renamed from R?; footprint Resistor_THT:R_Axial_DIN0204_L3.6mm_D1.6mm_P1.90mm_Vertical -> Resistor_SMD:R_0805_2012Metric_Pad1.20x1.40mm_HandSolder; Link (none) -> https://ro.mouser.com/ProductDetail/YAGEO/RC0805FR-071KL?qs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; Mfr. No. (none) -> RC0805FR-071KL
- R7: renamed from R23; footprint Resistor_THT:R_Axial_DIN0204_L3.6mm_D1.6mm_P1.90mm_Vertical -> Resistor_SMD:R_0805_2012Metric_Pad1.20x1.40mm_HandSolder; Link (none) -> https://ro.mouser.com/ProductDetail/YAGEO/AC0805FR-07470RL?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; Mfr. No. (none) -> AC0805FR-07470RL
- R8: renamed from R24; footprint Resistor_THT:R_Axial_DIN0204_L3.6mm_D1.6mm_P1.90mm_Vertical -> Resistor_SMD:R_0805_2012Metric_Pad1.20x1.40mm_HandSolder; Link (none) -> https://ro.mouser.com/ProductDetail/Vishay-Dale/CRCW080510K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; Mfr. No. (none) -> CRCW080510K0FKEAC
- RV1: footprint Potentiometer_THT:Potentiometer_Piher_PT-10-V10_Vertical -> Potentiometer_THT:Potentiometer_Piher_PT-6-V_Vertical
- SW1, SW2: renamed from SW?; footprint Button_Switch_THT:SW_PUSH_6mm -> Button_Switch_THT:SW_PUSH-12mm
- SW3: renamed from SW?; Link (none) -> https://ro.mouser.com/ProductDetail/Bourns/PEC11H-4220F-S00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; Mfr. No. (none) -> PEC11H-4220F-S0024
- U3: renamed from U?; footprint digikey-footprints:TO-220-3 -> Package_TO_SOT_SMD:TO-252-3_TabPin4; Link (none) -> https://ro.mouser.com/ProductDetail/onsemi/NCV7805BDTRKG?qs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; Mfr. No. (none) -> NCV7805BDTRKG
- U4: renamed from U?; Link (none) -> https://ro.mouser.com/ProductDetail/onsemi-Fairchild/FST325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; Mfr. No. (none) -> FST3253MTCX
- U5: renamed from U?; footprint Package_DIP:DIP-8_W7.62mm_LongPads -> Package_SO:SOIC-8_3.9x4.9mm_P1.27mm; Link (none) -> https://ro.mouser.com/ProductDetail/Texas-Instruments/LM456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; Mfr. No. (none) -> LM4562MAX/NOPB
- U6: renamed from U?; footprint Package_DIP:DIP-14_W7.62mm_LongPads -> Package_SO:SOIC-14_3.9x8.7mm_P1.27mm; Link (none) -> https://ro.mouser.com/ProductDetail/Texas-Instruments/SN74A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; Mfr. No. (none) -> SN74AC00D
- U8: renamed from U2; footprint Package_DIP:DIP-28_W7.62mm_Socket_LongPads -> Package_QFP:TQFP-32_7x7mm_P0.8mm; Link (none) -> https://ro.mouser.com/ProductDetail/Microchip-Technology-At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; Mfr. No. (none) -> ATMEGA328P-AN
- Y1: renamed from Y?; Link (none) -> https://ro.mouser.com/ProductDetail/Murata-Electronics/XRCG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; Mfr. No. (none) -> XRCGB27M000F2P01R0
- Y2: renamed from Y1; Link (none) -> https://ro.mouser.com/ProductDetail/ABRACON/ABLS-20000MHZ-2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; Mfr. No. (none) -> ABLS-20.000MHZ-20-B-3-H-T
- gave numbers to parts that had none: 1
- renumbered U8 to U2, U3 to U7
Connections:
- net +12V: no longer U7.15 (A/VEE)
- net +5V: now also C29.1, C6.1, C7.1, L3.1, RV1.1, U7.15 (A/VEE), U7.2 (VDD), U8.7 (VCC); no longer C4.1, C5.1, U3.3 (OUT)
- net RF_SIGNAL: now also U2.1 (RF_IN_1), U2.2 (RF_IN_2)
- new net: C4.1, C5.1, L1.1, U3.3 (OUT)
- no-connect marks 8 -> 12
Other:
- moved on the sheet: C1, C14, C17, C18, C2, C20, C21, C23, C24, C25, C26, C27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
