File: Hardware/uSDX_BPF/uSDX_BPF.kicad_sch (KiCad schematic)
At the start: 18 parts, among them P1 GND, P2 GND, P3 ANT2, P4 ANT1, P5 +12V, P6 TX, P7 RX, P8 GND

Commit message: updated the project with transferrable libraries
Parts:
- C1, C2, C3, C4, C5, C6: footprint Capacitor_THT:C_Disc_D3.0mm_W1.6mm_P2.50mm -> user_footprints:C_Disc_D3.0mm_W1.6mm_P2.50mm
- L1, L2, L3, L4: footprint Inductor_THT:L_Toroid_Vertical_L10.0mm_W5.0mm_P5.08mm -> user_footprints:L_Toroid_Vertical_L10.0mm_W5.0mm_P5.08mm
Changed lines of the file:
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@@
       (effects (font (size 1.27 1.27)) (justify left))
     )
-    (property "Footprint" "Capacitor_THT:C_Disc_D3.0mm_W1.6mm_P2.50mm" (id 2) (at 107.6452 100.33 0)
+    (property "Footprint" "user_footprints:C_Disc_D3.0mm_W1.6mm_P2.50mm" (id 2) (at 107.6452 100.33 0)
       (effects (font (size 1.27 1.27)) hide)
     )
@@
       (effects (font (size 1.27 1.27)) (justify left))
     )
-    (property "Footprint" "Capacitor_THT:C_Disc_D3.0mm_W1.6mm_P2.50mm" (id 2) (at 120.3452 100.33 0)
+    (property "Footprint" "user_footprints:C_Disc_D3.0mm_W1.6mm_P2.50mm" (id 2) (at 120.3452 100.33 0)
       (effects (font (size 1.27 1.27)) hide)
     )
@@
     (property "Reference" "L1" (id 0) (at 113.03 84.455 90))
     (property "Value" "T37-6 (16T)" (id 1) (at 113.03 86.7664 90))
-    (property "Footprint" "Inductor_THT:L_Toroid_Vertical_L10.0mm_W5.0mm_P5.08mm" (id 2) (at 113.03 90.17 0)
+    (property "Footprint" "user_footprints:L_Toroid_Vertical_L10.0mm_W5.0mm_P5.08mm" (id 2) (at 113.03 90.17 0)
       (effects (font (size 1.27 1.27)) hide)
     )
@@
       (effects (font (size 1.27 1.27)) (justify left))
     )
-    (property "Footprint" "Capacitor_THT:C_Disc_D3.0mm_W1.6mm_P2.50mm" (id 2) (at 133.0452 100.33 0)
+    (property "Footprint" "user_footprints:C_Disc_D3.0mm_W1.6mm_P2.50mm" (id 2) (at 133.0452 100.33 0)
       (effects (font (size 1.27 1.27)) hide)
     )
@@
     (property "Reference" "L2" (id 0) (at 125.73 84.455 90))
     (property "Value" "T37-6 (17T)" (id 1) (at 125.73 86.7664 90))
-    (property "Footprint" "Inductor_THT:L_Toroid_Vertical_L10.0mm_W5.0mm_P5.08mm" (id 2) (at 125.73 90.17 0)
+    (property "Footprint" "user_footprints:L_Toroid_Vertical_L10.0mm_W5.0mm_P5.08mm" (id 2) (at 125.73 90.17 0)
       (effects (font (size 1.27 1.27)) hide)
     )
@@
       (effects (font (size 1.27 1.27)) (justify left))
     )
-    (property "Footprint" "Capacitor_THT:C_Disc_D3.0mm_W1.6mm_P2.50mm" (id 2) (at 145.7452 100.33 0)
+    (property "Footprint" "user_footprints:C_Disc_D3.0mm_W1.6mm_P2.50mm" (id 2) (at 145.7452 100.33 0)
       (effects (font (size 1.27 1.27)) hide)
     )
@@
     (property "Reference" "L3" (id 0) (at 138.43 84.455 90))
     (property "Value" "T37-6 (16T)" (id 1) (at 138.43 86.7664 90))
-    (property "Footprint" "Inductor_THT:L_Toroid_Vertical_L10.0mm_W5.0mm_P5.08mm" (id 2) (at 138.43 90.17 0)
+    (property "Footprint" "user_footprints:L_Toroid_Vertical_L10.0mm_W5.0mm_P5.08mm" (id 2) (at 138.43 90.17 0)
       (effects (font (size 1.27 1.27)) hide)
     )
@@
     (property "Reference" "C5" (id 0) (at 162.56 83.7692 90))
     (property "Value" "100nF" (id 1) (at 162.56 86.0806 90))
-    (property "Footprint" "Capacitor_THT:C_Disc_D3.0mm_W1.6mm_P2.50mm" (id 2) (at 158.75 91.1352 0)
+    (property "Footprint" "user_footprints:C_Disc_D3.0mm_W1.6mm_P2.50mm" (id 2) (at 158.75 91.1352 0)
       (effects (font (size 1.27 1.27)) hide)
     )
@@
       (effects (font (size 1.27 1.27)) (justify left))
     )
-    (property "Footprint" "Capacitor_THT:C_Disc_D3.0mm_W1.6mm_P2.50mm" (id 2) (at 169.8752 100.33 0)
+    (property "Footprint" "user_footprints:C_Disc_D3.0mm_W1.6mm_P2.50mm" (id 2) (at 169.8752 100.33 0)
       (effects (font (size 1.27 1.27)) hide)
     )
@@
     (property "Reference" "L4" (id 0) (at 177.8 81.915 90))
     (property "Value" "T50-2 (9T)" (id 1) (at 177.8 84.2264 90))
-    (property "Footprint" "Inductor_THT:L_Toroid_Vertical_L10.0mm_W5.0mm_P5.08mm" (id 2) (at 177.8 87.63 0)
+    (property "Footprint" "user_footprints:L_Toroid_Vertical_L10.0mm_W5.0mm_P5.08mm" (id 2) (at 177.8 87.63 0)
       (effects (font (size 1.27 1.27)) hide)
     )
@@
     )
     (path "/00000000-0000-0000-0000-000061c8d39b"
-      (reference "C1") (unit 1) (value "180pF") (footprint "Capacitor_THT:C_Disc_D3.0mm_W1.6mm_P2.50mm")
+      (reference "C1") (unit 1) (value "180pF") (footprint "user_footprints:C_Disc_D3.0mm_W1.6mm_P2.50mm")
     )
     (path "/00000000-0000-0000-0000-000061c8db67"
-      (reference "C2") (unit 1) (value "390pF") (footprint "Capacitor_THT:C_Disc_D3.0mm_W1.6mm_P2.50mm")
+      (reference "C2") (unit 1) (value "390pF") (footprint "user_footprints:C_Disc_D3.0mm_W1.6mm_P2.50mm")
     )
     (path "/00000000-0000-0000-0000-000061c904bf"
-      (reference "C3") (unit 1) (value "390pF") (footprint "Capacitor_THT:C_Disc_D3.0mm_W1.6mm_P2.50mm")
+      (reference "C3") (unit 1) (value "390pF") (footprint "user_footprints:C_Disc_D3.0mm_W1.6mm_P2.50mm")
     )
     (path "/00000000-0000-0000-0000-000061c920d4"
-      (reference "C4") (unit 1) (value "180pF") (footprint "Capacitor_THT:C_Disc_D3.0mm_W1.6mm_P2.50mm")
+      (reference "C4") (unit 1) (value "180pF") (footprint "user_footprints:C_Disc_D3.0mm_W1.6mm_P2.50mm")
     )
     (path "/00000000-0000-0000-0000-000061c9700c"
-      (reference "C5") (unit 1) (value "100nF") (footprint "Capacitor_THT:C_Disc_D3.0mm_W1.6mm_P2.50mm")
+      (reference "C5") (unit 1) (value "100nF") (footprint "user_footprints:C_Disc_D3.0mm_W1.6mm_P2.50mm")
     )
     (path "/00000000-0000-0000-0000-000061c980c2"
-      (reference "C6") (unit 1) (value "30pF") (footprint "Capacitor_THT:C_Disc_D3.0mm_W1.6mm_P2.50mm")
+      (reference "C6") (unit 1) (value "30pF") (footprint "user_footprints:C_Disc_D3.0mm_W1.6mm_P2.50mm")
     )
     (path "/00000000-0000-0000-0000-000061c8e10c"
-      (reference "L1") (unit 1) (value "T37-6 (16T)") (footprint "Inductor_THT:L_Toroid_Vertical_L10.0mm_W5.0mm_P5.08mm")
+      (reference "L1") (unit 1) (value "T37-6 (16T)") (footprint "user_footprints:L_Toroid_Vertical_L10.0mm_W5.0mm_P5.08mm")
     )
     (path "/00000000-0000-0000-0000-000061c908f9"
-      (reference "L2") (unit 1) (value "T37-6 (17T)") (footprint "Inductor_THT:L_Toroid_Vertical_L10.0mm_W5.0mm_P5.08mm")
+      (reference "L2") (unit 1) (value "T37-6 (17T)") (footprint "user_footprints:L_Toroid_Vertical_L10.0mm_W5.0mm_P5.08mm")
     )
     (path "/00000000-0000-0000-0000-000061c9245e"
-      (reference "L3") (unit 1) (value "T37-6 (16T)") (footprint "Inductor_THT:L_Toroid_Vertical_L10.0mm_W5.0mm_P5.08mm")
+      (reference "L3") (unit 1) (value "T37-6 (16T)") (footprint "user_footprints:L_Toroid_Vertical_L10.0mm_W5.0mm_P5.08mm")
     )
     (path "/00000000-0000-0000-0000-000061c988b3"
-      (reference "L4") (unit 1) (value "T50-2 (9T)") (footprint "Inductor_THT:L_Toroid_Vertical_L10.0mm_W5.0mm_P5.08mm")
+      (reference "L4") (unit 1) (value "T50-2 (9T)") (footprint "user_footprints:L_Toroid_Vertical_L10.0mm_W5.0mm_P5.08mm")
     )
     (path "/00000000-0000-0000-0000-000061c89abd"
