File: Hardware/uSDX_SMD/uSDX_SMD.kicad_sch (KiCad schematic)
At the start: 104 parts, among them IC1 SI5351A-B-GTR, IC2 AZ1117CH, IC3 FST3253MTCX, IC4 MC74AC00DR2G, IC5 ATMEGA328P-ANR, J1 +12V, J2 CONSMA002-SMD-G-T, J3 Headphone_out, J4 SJ-43514-SMT-TR, J5 Conn_Coaxial, P1 DTR, P2 RX, P3 TX, P4 VIO, P5 CTS, P6 GND, Q1 BS170, Q2 BS170, Q3 BS170, Q4 BS170, Q5 BS170, SW1 RotaryEncoder, U1 LPF, U2 RC1602A, U3 LM4562, Y1 27MHz, Y2 20MHz

Commit message: updated the HW desigin and 3D models
Parts:
- Y2: footprint user_footprints:830108207209 -> SamacSys:830108207209
Connections:
- net at IC1.2 (XA): now also Y1.3; no longer Y1.2
Changed lines of the file:
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@@
     (property "Reference" "Y1" (id 0) (at 59.69 112.5728 0))
     (property "Value" "27MHz" (id 1) (at 59.69 114.8842 0))
-    (property "Footprint" "user_footprints:XRCGB27M000F2P01R0" (id 2) (at 59.69 119.38 0)
+    (property "Footprint" "user_footprints:XRCGB27M000F2P01R0" (id 2) (at 59.69 127 0)
       (effects (font (size 1.27 1.27)) hide)
     )
@@
     )
     (pin "1")
-    (pin "2")
+    (pin "3")
   )
   (symbol (lib_id "power:GND") (at 308.61 62.23 0) (unit 1)
@@
     (property "Reference" "Y2" (id 0) (at 429.26 97.79 0))
     (property "Value" "20MHz" (id 1) (at 431.8 97.79 0))
-    (property "Footprint" "user_footprints:830108207209" (id 2) (at 425.45 95.25 0)
+    (property "Footprint" "SamacSys:830108207209" (id 2) (at 425.45 95.25 0)
       (effects (font (size 1.27 1.27)) hide)
     )
@@
       (effects (font (size 1.27 1.27)) (justify left) hide)
     )
-    (pin "3")
-    (pin "2")
     (pin "1")
+    (pin "2")
+    (pin "3")
   )
   (symbol (lib_id "SamacSys_Parts:SJ-43514-SMT-TR") (at 201.93 39.37 0) (unit 1)
@@
     )
     (path "/00000000-0000-0000-0000-000061ca7442"
-      (reference "Y2") (unit 1) (value "20MHz") (footprint "user_footprints:830108207209")
+      (reference "Y2") (unit 1) (value "20MHz") (footprint "SamacSys:830108207209")
     )
   )

Commit message: updated the project with transferrable libraries
Parts:
- C1: footprint SamacSys_Parts:EEE0GA101SR -> user_footprints:EEE0GA101SR
- C10, C12, C13, C15, C16, C17, C18, C19, C2, C20, C21, C22, C23, C24, C25, C26, C27, C28, C29, C3, C30, C31, C32, C34, C4, C5, C6, C7, C8: footprint Capacitor_SMD:C_0805_2012Metric -> user_footprints:C_0805_2012Metric
- C11, C14, C33, C9: footprint SamacSys_Parts:CAPAE430X470N -> user_footprints:CAPAE430X470N
- D1: footprint SamacSys_Parts:SODFL4626X110N -> user_footprints:SODFL4626X110N
- D2, D3: footprint SamacSys_Parts:SOD3816X135N -> user_footprints:SOD3816X135N
- IC1: footprint SamacSys_Parts:SOP50P490X110-10N -> user_footprints:SOP50P490X110-10N
- IC3: footprint SamacSys_Parts:SOP65P640X110-16N -> user_footprints:SOP65P640X110-16N
- IC4: footprint SamacSys_Parts:SOIC127P600X175-14N -> user_footprints:SOIC127P600X175-14N
- IC5: footprint SamacSys_Parts:QFP80P900X900X120-32N -> user_footprints:QFP80P900X900X120-32N
- J2: footprint SamacSys:CONSMA002SMDGT -> user_footprints:CONSMA002SMDGT
- J3: footprint SamacSys_Parts:STX31503C1 -> user_footprints:STX31503C1
- J4: footprint SamacSys_Parts:SJ43514SMTTR -> user_footprints:SJ43514SMTTR
- R1, R10, R11, R12, R13, R14, R15, R16, R17, R18, R19, R2, R20, R21, R22, R23, R24, R25, R26, R28, R29, R3, R4, R5, R6, R7, R8, R9: footprint Resistor_SMD:R_0805_2012Metric -> user_footprints:R_0805_2012Metric
- S1, S2: footprint SamacSys_Parts:PTS125SM122LFS -> user_footprints:PTS125SM122LFS
- U3: footprint SamacSys_Parts:SOIC127P600X175-8N -> user_footprints:SOIC127P600X175-8N
- Y2: footprint SamacSys:830108207209 -> user_footprints:830108207209
