File: Hardware/uSDX_Transceiver_SMD/uSDX_Transceiver_SMD.sch (KiCad schematic (older format))
At the start: 104 parts, among them IC1 SI5351A-B-GTR, IC2 LM1117MPX-50NOPB, IC3 FST3253MTCX, IC4 MC74AC00DR2G, IC5 ATMEGA328P-ANR, J1 +12V, J2 CONSMA002-SMD-G-T, J3 Headphone_out, J4 SJ-43514-SMT-TR, P1 DTR, P2 RX, P3 TX, P4 VIO, P5 CTS, P6 GND, Q1 BS170, Q2 BS170, Q3 BS170, Q4 BS170, Q5 BS170, SW1 RotaryEncoder, U1 LPF, U2 RC1602A, U3 LM4562, Y1 27MHz, Y2 20MHz

Commit message: added tests for the LCD
Parts:
- C1: symbol SamacSys_Parts:EEE-FK1C101SR -> uSDX_Transceiver_SMD-rescue:EEE-FK1C101SR-SamacSys_Parts
- C10, C12, C13, C15, C16, C17, C18, C19, C2, C20, C21, C22, C23, C24, C25, C26, C27, C28, C29, C3, C30, C31, C32, C34, C4, C5, C6, C7, C8: symbol Device:C -> uSDX_Transceiver_SMD-rescue:C-Device
- C11, C14, C33, C9: symbol SamacSys_Parts:UCQ1C100MCL1GB -> uSDX_Transceiver_SMD-rescue:UCQ1C100MCL1GB-SamacSys_Parts
- D1: symbol SamacSys_Parts:1N4007F -> uSDX_Transceiver_SMD-rescue:1N4007F-SamacSys_Parts
- D2, D3: symbol SamacSys_Parts:1N4148W_R2_00001 -> uSDX_Transceiver_SMD-rescue:1N4148W_R2_00001-SamacSys_Parts
- IC1: symbol SamacSys_Parts:SI5351A-B-GTR -> uSDX_Transceiver_SMD-rescue:SI5351A-B-GTR-SamacSys_Parts
- IC2: symbol SamacSys_Parts:LM1117MPX-50NOPB -> uSDX_Transceiver_SMD-rescue:LM1117MPX-50NOPB-SamacSys_Parts
- IC3: symbol SamacSys_Parts:FST3253MTCX -> uSDX_Transceiver_SMD-rescue:FST3253MTCX-SamacSys_Parts
- IC4: symbol SamacSys_Parts:MC74AC00DR2G -> uSDX_Transceiver_SMD-rescue:MC74AC00DR2G-SamacSys_Parts
- IC5: symbol SamacSys_Parts:ATMEGA328P-ANR -> uSDX_Transceiver_SMD-rescue:ATMEGA328P-ANR-SamacSys_Parts
- J1: symbol SamacSys_Parts:16PJ200 -> uSDX_Transceiver_SMD-rescue:16PJ200-SamacSys_Parts
- J2: symbol SamacSys_Parts:CONSMA002-SMD-G-T -> uSDX_Transceiver_SMD-rescue:CONSMA002-SMD-G-T-SamacSys_Parts
- J3: symbol SamacSys_Parts:STX-3150-3C-1 -> uSDX_Transceiver_SMD-rescue:STX-3150-3C-1-SamacSys_Parts
- J4: symbol SamacSys_Parts:SJ-43514-SMT-TR -> uSDX_Transceiver_SMD-rescue:SJ-43514-SMT-TR-SamacSys_Parts
- L1, L2: symbol user:MSS6122-104MLC -> uSDX_Transceiver_SMD-rescue:MSS6122-104MLC-user
- P1, P2, P3, P4, P5, P6: symbol user:Pin -> uSDX_Transceiver_SMD-rescue:Pin-user
- Q1, Q2, Q3, Q4, Q5: symbol Device:Q_NMOS_DGS -> uSDX_Transceiver_SMD-rescue:Q_NMOS_DGS-Device
- R1, R10, R11, R12, R13, R14, R15, R16, R17, R18, R19, R2, R20, R21, R22, R23, R24, R25, R26, R27, R28, R29, R3, R4, R5, R6, R7, R8, R9: symbol Device:R -> uSDX_Transceiver_SMD-rescue:R-Device
- RV1: symbol Device:R_Potentiometer_Trim -> uSDX_Transceiver_SMD-rescue:R_Potentiometer_Trim-Device
- S1, S2, S3: symbol SamacSys_Parts:PTS125SM122LFS -> uSDX_Transceiver_SMD-rescue:PTS125SM122LFS-SamacSys_Parts
- SW1: symbol Device:RotaryEncoder_Switch -> uSDX_Transceiver_SMD-rescue:RotaryEncoder_Switch-Device
- TP1, TP2, TP3, TP4, TP5, TP6: symbol user:testpoint -> uSDX_Transceiver_SMD-rescue:testpoint-user
- U1: symbol user:LPF -> uSDX_Transceiver_SMD-rescue:LPF-user
- U2: symbol user:RC1602A -> uSDX_Transceiver_SMD-rescue:RC1602A-user
- U3: symbol user:LM4562 -> uSDX_Transceiver_SMD-rescue:LM4562-user
- Y1, Y2: symbol Device:Crystal -> uSDX_Transceiver_SMD-rescue:Crystal-Device
